Commit message: added

File: src/bot_description/urdf/mybot.xacro (robot description, xacro)
@@ -2,7 +2,7 @@
 <robot name="mybot" xmlns:xacro="http://www.ros.org/wiki/xacro">
 <!-- Include the Xacro files -->
-  <xacro:include filename="$(find bot_design)/urdf/materials.xacro" />
-  <xacro:include filename="$(find bot_design)/urdf/gazebo.xacro" />
-  <xacro:include filename="$(find bot_design)/urdf/macro.xacro" />
+  <xacro:include filename="$(find bot_description)/urdf/materials.xacro" />
+  <xacro:include filename="$(find bot_description)/urdf/mybot.gazebo" />
+  <xacro:include filename="$(find bot_description)/urdf/macro.xacro" />
  <!-- chassis definition -->
   <link name="link_chassis">
@@ -22,5 +22,5 @@
       <origin rpy="0 0 0" xyz="0 0 0"/>
       <geometry>
-        <cylinder length="0.05" radius="0.5"/>
+        <cylinder length="0.05" radius="0.3"/>
       </geometry>
       <material name="blue"/>

Commit message: added

File: src/bot_description/urdf/mybot.xacro (robot description, xacro)
@@ -22,5 +22,5 @@
       <origin rpy="0 0 0" xyz="0 0 0"/>
       <geometry>
-        <cylinder length="0.05" radius="0.3"/>
+        <cylinder length="0.05" radius="0.5"/>
       </geometry>
       <material name="blue"/>
